File: v1.2/Kicad Files/A314v1.2.kicad_pcb (KiCad board)
At the start: 4 copper layers, 75 x 89 mm, 107 parts, among them IC1 SN74CBT16244CDL, IC10 24AA32ASN, IC11 TPS63020DSJR, IC2 SN74CBT16244CDL, IC3 SN74CBT16244CDL, IC4 IS61WV51216BLL-10TLI, IC5 10M08SCE144, IC6 DS3231M, IC8 NB3N502, IC9 TPS77033, T1 2N4401

Commit message: More cleanup
Parts:
- removed GND0, UNK3V3, UNK4V3, UNK5V0: TPPAD1-13, A314v1.2:P1-13
- removed U$1: , A314v1.2:OSHW_8_NOTEXT
- removed U$2, U$3: , A314v1.2:A314_LOGO
- removed U$4: , A314v1.2:OSHW_8MM
- C1, C11, C12, C13, C14, C15, C19, C20, C21, C22, C23, C24, C3, C31, C32, C33, C34, C4, C41, C42, C50, C51, C52, C53, C54, C55, C56, C57, C58, C59, C60, C61, C62, C63, C64, C65, C66, C67, C68, C69, C7, C70, C71, C72, C8, C9: footprint A314v1.2:C0805 -> Capacitor_SMD:C_0805_2012Metric_Pad1.18x1.45mm_HandSolder
- C10, C16, C17, C18, C2, C5, C6: footprint A314v1.2:C1812K -> Capacitor_SMD:C_1812_4532Metric_Pad1.57x3.40mm_HandSolder
- IC10: value 24AA32ASN -> 24SN
- IC7: value (none) -> TPS565208DDC
- IC9: value TPS77033 -> TPS770
- JMP2, JMPB3: value (none) -> JP1E
- R1, R10, R15, R16, R17, R18, R19, R2, R20, R21, R22, R3, R4, R5, R6, R7, R8, R9: footprint A314v1.2:R0805 -> Resistor_SMD:R_0805_2012Metric_Pad1.20x1.40mm_HandSolder
- RASP_I2C0: value (none) -> MA04-1
Connections:
- net + renamed Net-(IC6-VBAT)
- net +3V3 renamed +3.3V
- net +5V/1 renamed +5V/1
- net 14MHZ renamed Net-(IC5C-GPIO26/CLK0N)
- net A2 renamed /AMIGA Interface/A2
- net A3 renamed /AMIGA Interface/A3
- net A4 renamed /AMIGA Interface/A4
- net A5 renamed /AMIGA Interface/A5
- net BST1 renamed Net-(IC7-VBST)
- net CFG_DNE renamed Net-(IC5I-GPIO138/CONF_DONE)
- net CFG_SEL renamed Net-(IC5I-GPIO126/CONFIG_SEL)
- net CLKRD renamed /AMIGA Interface/CLKRD
- net CLKWR renamed /AMIGA Interface/CLKWR
- net D0 renamed /AMIGA Interface/D0
- net D1 renamed /AMIGA Interface/D1
- net D2 renamed /AMIGA Interface/D2
- net D3 renamed /AMIGA Interface/D3
- net DRA0 renamed /AMIGA Interface/DRA0
- net DRA1 renamed /AMIGA Interface/DRA1
- net DRA2 renamed /AMIGA Interface/DRA2
- net DRA3 renamed /AMIGA Interface/DRA3
- net DRA4 renamed /AMIGA Interface/DRA4
- net DRA5 renamed /AMIGA Interface/DRA5
- net DRA6 renamed /AMIGA Interface/DRA6
- net DRA7 renamed /AMIGA Interface/DRA7
- net DRA8 renamed /AMIGA Interface/DRA8
- net DRA8_L renamed Net-(IC1D-B4)
- net DRAS0 renamed /AMIGA Interface/DRAS0
- net DRAS0_L renamed Net-(IC1D-B1)
- net DRAS1 renamed /AMIGA Interface/DRAS1
- net DRAS1_L renamed Net-(IC1C-B4)
- net DRCASL renamed /AMIGA Interface/DRCASL
- net DRCASL_L renamed Net-(IC1D-B3)
- net DRCASU renamed /AMIGA Interface/DRCASU
- net DRCASU_L renamed Net-(IC1D-B2)
- net DRCCK renamed /AMIGA Interface/DRCCK
- net DRD0 renamed /AMIGA Interface/DRD0
- net DRD1 renamed /AMIGA Interface/DRD1
- net DRD10 renamed /AMIGA Interface/DRD10
- net DRD11 renamed /AMIGA Interface/DRD11
- net DRD12 renamed /AMIGA Interface/DRD12
- net DRD13 renamed /AMIGA Interface/DRD13
- net DRD14 renamed /AMIGA Interface/DRD14
- net DRD15 renamed /AMIGA Interface/DRD15
- net DRD2 renamed /AMIGA Interface/DRD2
- net DRD3 renamed /AMIGA Interface/DRD3
- net DRD4 renamed /AMIGA Interface/DRD4
- net DRD5 renamed /AMIGA Interface/DRD5
- net DRD6 renamed /AMIGA Interface/DRD6
- net DRD7 renamed /AMIGA Interface/DRD7
- net DRD8 renamed /AMIGA Interface/DRD8
- net DRD9 renamed /AMIGA Interface/DRD9
- net DRWE renamed /AMIGA Interface/DRWE
- net DRWE_L renamed Net-(IC1C-B3)
- net FB1 renamed Net-(IC7-VFB)
- net FB2 renamed Net-(IC11-FB)
- net HAT_SCL renamed Net-(IC10-SCL)
- net HAT_SDA renamed Net-(IC10-SDA)
- net INT2A renamed Net-(IC3C-B4)
- net L1 renamed Net-(IC11-L1-Pad8)
- net L2 renamed Net-(IC11-L2-Pad6)
- net LB renamed /SRAM & RTC/LB
- net LED_CTRL renamed Net-(IC5I-GPIO123/VREFB8N0)
- net LED_PWR renamed Net-(LED0A-S)
- net LED_RTN renamed Net-(LED0B-S)
- net MISO renamed /Raspberry & DRAM Bus/MISO
- net MOSI renamed /Raspberry & DRAM Bus/MOSI
- net OE renamed /SRAM & RTC/OE
- net OUTPUT_EN renamed Net-(IC3D-~{OE})
- net PI_SCL renamed Net-(RP1-SCL)
- net PI_SDA renamed Net-(RP1-SDA)
- net RAS0 renamed Net-(IC1D-A1)
- net RAS1 renamed Net-(IC1C-A4)
- net SCL renamed Net-(IC5G-GPIO97/VREFB6N0)
- net SCLK renamed /Raspberry & DRAM Bus/SCLK
- net SDA renamed Net-(IC5H-GPIO112/VREFB7N0)
- net SRA0 renamed /SRAM & RTC/SRA0
- net SRA1 renamed /SRAM & RTC/SRA1
- net SRA12 renamed /SRAM & RTC/SRA12
- net SRA13 renamed /SRAM & RTC/SRA13
- net SRA14 renamed /SRAM & RTC/SRA14
- net SRA15 renamed /SRAM & RTC/SRA15
- net SRA16 renamed /SRAM & RTC/SRA16
- net SRA17 renamed /SRAM & RTC/SRA17
- net SRA18 renamed /SRAM & RTC/SRA18
- net SRA2 renamed /SRAM & RTC/SRA2
- net SRA3 renamed /SRAM & RTC/SRA3
- net SRA4 renamed /SRAM & RTC/SRA4
- net SRA5 renamed /SRAM & RTC/SRA5
- net SRA6 renamed /SRAM & RTC/SRA6
- net SRA7 renamed /SRAM & RTC/SRA7
- net SRA8 renamed /SRAM & RTC/SRA8
- net SRA9 renamed /SRAM & RTC/SRA9
- net SRD0 renamed /SRAM & RTC/SRD0
- net SRD1 renamed /SRAM & RTC/SRD1
- net SRD10 renamed /SRAM & RTC/SRD10
- net SRD11 renamed /SRAM & RTC/SRD11
- net SRD12 renamed /SRAM & RTC/SRD12
- net SRD13 renamed /SRAM & RTC/SRD13
- net SRD14 renamed /SRAM & RTC/SRD14
- net SRD15 renamed /SRAM & RTC/SRD15
- net SRD2 renamed /SRAM & RTC/SRD2
- net SRD3 renamed /SRAM & RTC/SRD3
- net SRD4 renamed /SRAM & RTC/SRD4
- net SRD5 renamed /SRAM & RTC/SRD5
- net SRD6 renamed /SRAM & RTC/SRD6
- net SRD7 renamed /SRAM & RTC/SRD7
- net SRD8 renamed /SRAM & RTC/SRD8
- net SRD9 renamed /SRAM & RTC/SRD9
- net SW renamed Net-(IC7-SW)
- net TCK renamed /Raspberry & DRAM Bus/TCK
- net TDI renamed /Raspberry & DRAM Bus/TDI
- net TDO renamed /Raspberry & DRAM Bus/TDO
- net TMS renamed /Raspberry & DRAM Bus/TMS
- net UB renamed /SRAM & RTC/UB
- net VCC/2 renamed +3V3_PI
- net VINA renamed Net-(IC11-EN)
- net WE renamed /SRAM & RTC/WE
- net WP renamed Net-(IC10-WP)
- net ~{CFG} renamed Net-(IC5I-GPI129/~{CONFIG})
- net ~{STAT} renamed Net-(IC5I-GPIO136/~{STATUS})
- CNY1 pad 32: EXRAM -> GND
- CNY1 pad 55: (no net) -> unconnected-(CNY1-+12V-Pad55)
- CNY1 pad 56: (no net) -> unconnected-(CNY1--12V-Pad56)
- IC11 pad 14: (no net) -> unconnected-(IC11-PG-Pad14)
- IC2 pad 46: (no net) -> unconnected-(IC2A-A2-Pad46)
- IC3 pad 16: (no net) -> unconnected-(IC3C-B3-Pad16)
- IC3 pad 19: (no net) -> unconnected-(IC3D-B1-Pad19)
- IC3 pad 20: (no net) -> unconnected-(IC3D-B2-Pad20)
- IC3 pad 22: (no net) -> unconnected-(IC3D-B3-Pad22)
- IC3 pad 23: (no net) -> unconnected-(IC3D-B4-Pad23)
- IC3 pad 26: (no net) -> unconnected-(IC3D-A4-Pad26)
- IC3 pad 27: (no net) -> unconnected-(IC3D-A3-Pad27)
- IC3 pad 29: (no net) -> unconnected-(IC3D-A2-Pad29)
- IC3 pad 30: (no net) -> unconnected-(IC3D-A1-Pad30)
- IC5 pad 17: (no net) -> unconnected-(IC5B-GPIO17/VREFB1N0-Pad17)
- IC5 pad 25: (no net) -> unconnected-(IC5B-GPIO25-Pad25)
- IC5 pad 27: (no net) -> unconnected-(IC5C-GPIO27/CLK0P-Pad27)
- IC5 pad 30: (no net) -> unconnected-(IC5C-GPIO30/VREFB2N0-Pad30)
- IC6 pad 1: (no net) -> unconnected-(IC6-32KHZ-Pad1)
- IC6 pad 3: (no net) -> unconnected-(IC6-~{INT}/SQW-Pad3)
- IC6 pad 4: (no net) -> unconnected-(IC6-~{RST}-Pad4)
- IC8 pad 4: (no net) -> unconnected-(IC8-CLKREF-Pad4)
- IC8 pad 8: (no net) -> unconnected-(IC8-X2-Pad8)
- IC9 pad 4: (no net) -> unconnected-(IC9-NC/FB-Pad4)
- JMP2 pad 2: EXRAM -> GND
- R12 pad 3: (no net) -> unconnected-(R12C-P$1-Pad3)
- R12 pad 4: (no net) -> unconnected-(R12D-P$1-Pad4)
- R12 pad 5: (no net) -> unconnected-(R12D-P$2-Pad5)
- R12 pad 6: (no net) -> unconnected-(R12C-P$2-Pad6)
- RP1 pad 10: (no net) -> unconnected-(RP1-RXD-Pad10)
- RP1 pad 12: (no net) -> unconnected-(RP1-GPIO18-Pad12)
- RP1 pad 18: (no net) -> unconnected-(RP1-GPIO24-Pad18)
- RP1 pad 26: (no net) -> unconnected-(RP1-CE1@0-Pad26)
- RP1 pad 29: (no net) -> unconnected-(RP1-GPIO05-Pad29)
- RP1 pad 31: (no net) -> unconnected-(RP1-GPIO06-Pad31)
- RP1 pad 32: (no net) -> unconnected-(RP1-GPIO12-Pad32)
- RP1 pad 33: (no net) -> unconnected-(RP1-GPIO13-Pad33)
- RP1 pad 35: (no net) -> unconnected-(RP1-MISO@1-Pad35)
- RP1 pad 36: (no net) -> unconnected-(RP1-CE0@1-Pad36)
- RP1 pad 37: (no net) -> unconnected-(RP1-GPIO26-Pad37)
- RP1 pad 38: (no net) -> unconnected-(RP1-MOSI@1-Pad38)
- RP1 pad 40: (no net) -> unconnected-(RP1-SCLK@1-Pad40)
- RP1 pad 7: (no net) -> unconnected-(RP1-GPIO04-Pad7)
- RP1 pad 8: (no net) -> unconnected-(RP1-TXD-Pad8)
Routing:
- net EXRAM: track 6.06 -> 0.00 mm
- net GND: track 253.2 -> 259.3 mm
