File: v1.2/Kicad Files/A314v1.2_2.kicad_sch (KiCad schematic)
At the start: 6 parts, among them IC4 IS61WV51216BLL-10TLI, IC5 10M08SCE144, IC6 DS3231M

Commit message: More cleanup
Parts:
- R3, R4: symbol A314v1.2-eagle-import:R-EU_R0805 -> Device:R
Changed lines of the file:
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@@
 	(wire
 		(pts
-			(xy 180.34 185.42) (xy 180.34 187.96)
+			(xy 180.34 185.42) (xy 180.34 189.23)
 		)
 		(stroke
@@
 		)
 	)
+	(wire
+		(pts
+			(xy 175.26 196.85) (xy 175.26 198.12)
+		)
+		(stroke
+			(width 0)
+			(type default)
+		)
+	)
 	(bus
 		(pts
@@
 	(wire
 		(pts
-			(xy 175.26 187.96) (xy 175.26 185.42)
+			(xy 160.02 66.04) (xy 160.02 68.58)
 		)
 		(stroke
-			(width 0.1524)
-			(type solid)
+			(width 0)
+			(type default)
 		)
 	)
 	(wire
 		(pts
-			(xy 160.02 66.04) (xy 160.02 68.58)
+			(xy 175.26 185.42) (xy 175.26 189.23)
 		)
 		(stroke
-			(width 0)
-			(type default)
+			(width 0.1524)
+			(type solid)
 		)
 	)
@@
 	(wire
 		(pts
+			(xy 180.34 196.85) (xy 180.34 198.12)
+		)
+		(stroke
+			(width 0)
+			(type default)
+		)
+	)
+	(wire
+		(pts
 			(xy 198.12 215.9) (xy 198.12 218.44)
 		)
@@
 	)
 	(symbol
-		(lib_id "A314v1.2-eagle-import:R-EU_R0805")
-		(at 175.26 193.04 90)
+		(lib_id "Device:R")
+		(at 175.26 193.04 180)
 		(unit 1)
 		(exclude_from_sim no)
@@
 		(dnp no)
 		(property "Reference" "R4"
-			(at 173.7614 196.85 0)
+			(at 179.07 194.5386 0)
 			(effects
 				(font
@@
 		)
 		(property "Value" "3k9"
-			(at 176.022 194.31 0)
+			(at 176.53 192.278 0)
 			(effects
 				(font
@@
 		)
 		(property "Footprint" "A314v1.2:R0805"
-			(at 175.26 193.04 0)
+			(at 175.26 193.04 90)
 			(effects
 				(font
@@
 			)
 		)
-		(property "Datasheet" ""
+		(property "Datasheet" "~"
 			(at 175.26 193.04 0)
 			(effects
@@
 			)
 		)
-		(property "Description" ""
+		(property "Description" "Resistor"
 			(at 175.26 193.04 0)
 			(effects
@@
 	)
 	(symbol
-		(lib_id "A314v1.2-eagle-import:R-EU_R0805")
-		(at 180.34 193.04 90)
+		(lib_id "Device:R")
+		(at 180.34 193.04 180)
 		(unit 1)
 		(exclude_from_sim no)
@@
 		(dnp no)
 		(property "Reference" "R3"
-			(at 178.8414 196.85 0)
+			(at 184.15 194.5386 0)
 			(effects
 				(font
@@
 		)
 		(property "Value" "3k9"
-			(at 181.102 194.31 0)
+			(at 181.61 192.278 0)
 			(effects
 				(font
@@
 		)
 		(property "Footprint" "A314v1.2:R0805"
-			(at 180.34 193.04 0)
+			(at 180.34 193.04 90)
 			(effects
 				(font
@@
 			)
 		)
-		(property "Datasheet" ""
+		(property "Datasheet" "~"
 			(at 180.34 193.04 0)
 			(effects
@@
 			)
 		)
-		(property "Description" ""
+		(property "Description" "Resistor"
 			(at 180.34 193.04 0)
 			(effects
