File: v1.2/Kicad Files/A314v1.2_3.kicad_sch (KiCad schematic)
At the start: 19 parts, among them IC10 24SN, IC5 10M08SCE144, IC8 NB3N502, T1 2N4401

Commit message: More cleanup
Parts:
- R10, R15, R16, R17, R18, R19, R22, R5, R6, R7, R8, R9: symbol A314v1.2-eagle-import:R-EU_R0805 -> Device:R
