File: v1.2/Kicad Files/A314v1.2_4.kicad_sch (KiCad schematic)
At the start: 71 parts, among them IC1 SN74CBT16244CDL, IC11 TPS63020DSJR, IC2 SN74CBT16244CDL, IC3 SN74CBT16244CDL, IC4 IS61WV51216BLL-10TLI, IC5 10M08SCE144, IC7 TPS565208DDC, IC9 TPS770

Commit message: More cleanup
Parts:
- C1, C11, C12, C13, C14, C15, C19, C20, C21, C22, C23, C24, C3, C31, C32, C33, C34, C4, C41, C42, C50, C51, C52, C53, C54, C55, C56, C57, C58, C59, C60, C61, C62, C63, C64, C65, C66, C67, C68, C69, C7, C70, C71, C72, C8, C9: footprint A314v1.2:C0805 -> Capacitor_SMD:C_0805_2012Metric_Pad1.18x1.45mm_HandSolder; symbol A314v1.2-eagle-import:C-EUC0805 -> Device:C
- C10, C16, C17, C18, C2, C5, C6: footprint A314v1.2:C1812K -> Capacitor_SMD:C_1812_4532Metric_Pad1.57x3.40mm_HandSolder
- R1, R2, R20, R21: symbol A314v1.2-eagle-import:R-EU_R0805 -> Device:R
